File: esp32-c6.kicad_sch (KiCad schematic)
At the start: 29 parts, among them J3 u.FL, U4 ESP32-C6FH8, Y1 40MHz

Commit message: updates
Parts:
- renumbered J3 to J1, R14 to R10, R15 to R11, R16 to R12, R6 to R2, R7 to R3, R8 to R4, R9 to R5, R10 to R6, R11 to R7, R12 to R8, R13 to R9, U4 to U3
Changed lines of the file:
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@@
 		(dnp no)
 		(fields_autoplaced yes)
-		(property "Reference" "R10"
+		(property "Reference" "R6"
 			(at 148.59 95.25 90)
 			(show_name no)
@@
 			(project "Overkill-core"
 				(path "/fc53a0b2-7a4c-469b-8f54-4e370debb709/b418b60c-f580-4941-9de1-4c275543c012/0d515c06-80db-41d9-898c-66653a1c38b5"
-					(reference "R10")
+					(reference "R6")
 					(unit 1)
 				)
@@
 		(dnp no)
 		(fields_autoplaced yes)
-		(property "Reference" "#PWR016"
+		(property "Reference" "#PWR010"
 			(at 196.85 58.42 0)
 			(hide yes)
@@
 			(project "Overkill-core"
 				(path "/fc53a0b2-7a4c-469b-8f54-4e370debb709/b418b60c-f580-4941-9de1-4c275543c012/0d515c06-80db-41d9-898c-66653a1c38b5"
-					(reference "#PWR016")
+					(reference "#PWR010")
 					(unit 1)
 				)
@@
 		(in_pos_files yes)
 		(dnp no)
-		(property "Reference" "R8"
+		(property "Reference" "R4"
 			(at 138.43 94.742 90)
 			(show_name no)
@@
 			(project "Overkill-core"
 				(path "/fc53a0b2-7a4c-469b-8f54-4e370debb709/b418b60c-f580-4941-9de1-4c275543c012/0d515c06-80db-41d9-898c-66653a1c38b5"
-					(reference "R8")
+					(reference "R4")
 					(unit 1)
 				)
@@
 		(dnp no)
 		(fields_autoplaced yes)
-		(property "Reference" "R13"
+		(property "Reference" "R9"
 			(at 158.75 105.41 90)
 			(show_name no)
@@
 			(project "Overkill-core"
 				(path "/fc53a0b2-7a4c-469b-8f54-4e370debb709/b418b60c-f580-4941-9de1-4c275543c012/0d515c06-80db-41d9-898c-66653a1c38b5"
-					(reference "R13")
+					(reference "R9")
 					(unit 1)
 				)
@@
 		(dnp no)
 		(fields_autoplaced yes)
-		(property "Reference" "R12"
+		(property "Reference" "R8"
 			(at 153.67 100.33 90)
 			(show_name no)
@@
 			(project "Overkill-core"
 				(path "/fc53a0b2-7a4c-469b-8f54-4e370debb709/b418b60c-f580-4941-9de1-4c275543c012/0d515c06-80db-41d9-898c-66653a1c38b5"
-					(reference "R12")
+					(reference "R8")
 					(unit 1)
 				)
@@
 		(dnp yes)
 		(fields_autoplaced yes)
-		(property "Reference" "R15"
+		(property "Reference" "R11"
 			(at 191.77 36.83 90)
 			(show_name no)
@@
 			(project "Overkill-core"
 				(path "/fc53a0b2-7a4c-469b-8f54-4e370debb709/b418b60c-f580-4941-9de1-4c275543c012/0d515c06-80db-41d9-898c-66653a1c38b5"
-					(reference "R15")
+					(reference "R11")
 					(unit 1)
 				)
@@
 		(dnp no)
 		(fields_autoplaced yes)
-		(property "Reference" "#PWR012"
+		(property "Reference" "#PWR06"
 			(at 57.15 53.34 0)
 			(hide yes)
@@
 			(project "Overkill-core"
 				(path "/fc53a0b2-7a4c-469b-8f54-4e370debb709/b418b60c-f580-4941-9de1-4c275543c012/0d515c06-80db-41d9-898c-66653a1c38b5"
-					(reference "#PWR012")
+					(reference "#PWR06")
 					(unit 1)
 				)
@@
 		(dnp no)
 		(fields_autoplaced yes)
-		(property "Reference" "R9"
+		(property "Reference" "R5"
 			(at 143.51 97.79 90)
 			(show_name no)
@@
 			(project "Overkill-core"
 				(path "/fc53a0b2-7a4c-469b-8f54-4e370debb709/b418b60c-f580-4941-9de1-4c275543c012/0d515c06-80db-41d9-898c-66653a1c38b5"
-					(reference "R9")
+					(reference "R5")
 					(unit 1)
 				)
@@
 		(dnp no)
 		(fields_autoplaced yes)
-		(property "Reference" "#PWR013"
+		(property "Reference" "#PWR07"
 			(at 90.17 124.46 0)
 			(hide yes)
@@
 			(project "Overkill-core"
 				(path "/fc53a0b2-7a4c-469b-8f54-4e370debb709/b418b60c-f580-4941-9de1-4c275543c012/0d515c06-80db-41d9-898c-66653a1c38b5"
-					(reference "#PWR013")
+					(reference "#PWR07")
 					(unit 1)
 				)
@@
 		(dnp no)
 		(fields_autoplaced yes)
-		(property "Reference" "R6"
+		(property "Reference" "R2"
 			(at 36.83 58.4199 0)
 			(show_name no)
@@
 			(project "Overkill-core"
 				(path "/fc53a0b2-7a4c-469b-8f54-4e370debb709/b418b60c-f580-4941-9de1-4c275543c012/0d515c06-80db-41d9-898c-66653a1c38b5"
-					(reference "R6")
+					(reference "R2")
 					(unit 1)
 				)
@@
 		(dnp no)
 		(fields_autoplaced yes)
-		(property "Reference" "R11"
+		(property "Reference" "R7"
 			(at 148.59 102.87 90)
 			(show_name no)
@@
 			(project "Overkill-core"
 				(path "/fc53a0b2-7a4c-469b-8f54-4e370debb709/b418b60c-f580-4941-9de1-4c275543c012/0d515c06-80db-41d9-898c-66653a1c38b5"
-					(reference "R11")
+					(reference "R7")
 					(unit 1)
 				)
@@
 		(dnp no)
 		(fields_autoplaced yes)
-		(property "Reference" "#PWR011"
+		(property "Reference" "#PWR05"
 			(at 34.29 77.47 0)
 			(hide yes)
@@
 			(project "Overkill-core"
 				(path "/fc53a0b2-7a4c-469b-8f54-4e370debb709/b418b60c-f580-4941-9de1-4c275543c012/0d515c06-80db-41d9-898c-66653a1c38b5"
-					(reference "#PWR011")
+					(reference "#PWR05")
 					(unit 1)
 				)
@@
 		(dnp no)
 		(fields_autoplaced yes)
-		(property "Reference" "U4"
+		(property "Reference" "U3"
 			(at 92.3133 116.84 0)
 			(show_name no)
@@
 			(project "Overkill-core"
 				(path "/fc53a0b2-7a4c-469b-8f54-4e370debb709/b418b60c-f580-4941-9de1-4c275543c012/0d515c06-80db-41d9-898c-66653a1c38b5"
-					(reference "U4")
+					(reference "U3")
 					(unit 1)
 				)
@@
 		(in_pos_files yes)
 		(dnp no)
-		(property "Reference" "R7"
+		(property "Reference" "R3"
 			(at 127 59.182 90)
 			(show_name no)
@@
 			(project "Overkill-core"
 				(path "/fc53a0b2-7a4c-469b-8f54-4e370debb709/b418b60c-f580-4941-9de1-4c275543c012/0d515c06-80db-41d9-898c-66653a1c38b5"
-					(reference "R7")
+					(reference "R3")
 					(unit 1)
 				)
@@
 		(dnp no)
 		(fields_autoplaced yes)
-		(property "Reference" "R16"
+		(property "Reference" "R12"
 			(at 199.39 36.8299 0)
 			(show_name no)
@@
 			(project "Overkill-core"
 				(path "/fc53a0b2-7a4c-469b-8f54-4e370debb709/b418b60c-f580-4941-9de1-4c275543c012/0d515c06-80db-41d9-898c-66653a1c38b5"
-					(reference "R16")
+					(reference "R12")
 					(unit 1)
 				)
@@
 		(dnp yes)
 		(fields_autoplaced yes)
-		(property "Reference" "R14"
+		(property "Reference" "R10"
 			(at 187.96 67.31 90)
 			(show_name no)
@@
 			(project "Overkill-core"
 				(path "/fc53a0b2-7a4c-469b-8f54-4e370debb709/b418b60c-f580-4941-9de1-4c275543c012/0d515c06-80db-41d9-898c-66653a1c38b5"
-					(reference "R14")
+					(reference "R10")
 					(unit 1)
 				)
@@
 		(dnp no)
 		(fields_autoplaced yes)
-		(property "Reference" "#PWR014"
+		(property "Reference" "#PWR08"
 			(at 128.27 55.88 0)
 			(hide yes)
@@
 			(project "Overkill-core"
 				(path "/fc53a0b2-7a4c-469b-8f54-4e370debb709/b418b60c-f580-4941-9de1-4c275543c012/0d515c06-80db-41d9-898c-66653a1c38b5"
-					(reference "#PWR014")
+					(reference "#PWR08")
 					(unit 1)
 				)
@@
 		(in_pos_files yes)
 		(dnp no)
-		(property "Reference" "J3"
+		(property "Reference" "J1"
 			(at 173.99 42.2031 0)
 			(show_name no)
@@
 			(project "Overkill-core"
 				(path "/fc53a0b2-7a4c-469b-8f54-4e370debb709/b418b60c-f580-4941-9de1-4c275543c012/0d515c06-80db-41d9-898c-66653a1c38b5"
-					(reference "J3")
+					(reference "J1")
 					(unit 1)
 				)
@@
 		(dnp no)
 		(fields_autoplaced yes)
-		(property "Reference" "#PWR015"
+		(property "Reference" "#PWR09"
 			(at 187.96 99.06 0)
 			(hide yes)
@@
 			(project "Overkill-core"
 				(path "/fc53a0b2-7a4c-469b-8f54-4e370debb709/b418b60c-f580-4941-9de1-4c275543c012/0d515c06-80db-41d9-898c-66653a1c38b5"
-					(reference "#PWR015")
-					(unit 1)
-				)
+					(reference "#PWR09")
+					(unit 1)
+				)
