File: esp32-p4.kicad_sch (KiCad schematic)
At the start: 46 parts, among them U5 ESP32-P4NRW32X, U6 W25Q128JVS, Y2 40MHz, Y3 32.768KHz

Commit message: updates
Parts:
- renumbered R17 to R13, R18 to R14, R19 to R15, R20 to R16, R21 to R17, R22 to R18, U5 to U4, U6 to U5
Changed lines of the file:
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@@
 		(dnp no)
 		(fields_autoplaced yes)
-		(property "Reference" "#PWR031"
+		(property "Reference" "#PWR025"
 			(at 266.7 53.34 0)
 			(hide yes)
@@
 			(project "Overkill-core"
 				(path "/fc53a0b2-7a4c-469b-8f54-4e370debb709/b418b60c-f580-4941-9de1-4c275543c012/c2c849f9-72ec-481b-977e-253b138385b2"
-					(reference "#PWR031")
+					(reference "#PWR025")
 					(unit 1)
 				)
@@
 		(dnp no)
 		(fields_autoplaced yes)
-		(property "Reference" "U6"
+		(property "Reference" "U5"
 			(at 267.97 139.6999 0)
 			(show_name no)
@@
 			(project "Overkill-core"
 				(path "/fc53a0b2-7a4c-469b-8f54-4e370debb709/b418b60c-f580-4941-9de1-4c275543c012/c2c849f9-72ec-481b-977e-253b138385b2"
-					(reference "U6")
+					(reference "U5")
 					(unit 1)
 				)
@@
 		(dnp no)
 		(fields_autoplaced yes)
-		(property "Reference" "#PWR022"
+		(property "Reference" "#PWR016"
 			(at 99.06 177.8 0)
 			(hide yes)
@@
 			(project "Overkill-core"
 				(path "/fc53a0b2-7a4c-469b-8f54-4e370debb709/b418b60c-f580-4941-9de1-4c275543c012/c2c849f9-72ec-481b-977e-253b138385b2"
-					(reference "#PWR022")
+					(reference "#PWR016")
 					(unit 1)
 				)
@@
 		(dnp no)
 		(fields_autoplaced yes)
-		(property "Reference" "#PWR024"
+		(property "Reference" "#PWR018"
 			(at 161.29 144.78 0)
 			(hide yes)
@@
 			(project "Overkill-core"
 				(path "/fc53a0b2-7a4c-469b-8f54-4e370debb709/b418b60c-f580-4941-9de1-4c275543c012/c2c849f9-72ec-481b-977e-253b138385b2"
-					(reference "#PWR024")
+					(reference "#PWR018")
 					(unit 1)
 				)
@@
 		(dnp no)
 		(fields_autoplaced yes)
-		(property "Reference" "R18"
+		(property "Reference" "R14"
 			(at 46.99 140.9699 0)
 			(show_name no)
@@
 			(project "Overkill-core"
 				(path "/fc53a0b2-7a4c-469b-8f54-4e370debb709/b418b60c-f580-4941-9de1-4c275543c012/c2c849f9-72ec-481b-977e-253b138385b2"
-					(reference "R18")
+					(reference "R14")
 					(unit 1)
 				)
@@
 		(dnp no)
 		(fields_autoplaced yes)
-		(property "Reference" "#PWR018"
+		(property "Reference" "#PWR012"
 			(at 27.94 96.52 0)
 			(hide yes)
@@
 			(project "Overkill-core"
 				(path "/fc53a0b2-7a4c-469b-8f54-4e370debb709/b418b60c-f580-4941-9de1-4c275543c012/c2c849f9-72ec-481b-977e-253b138385b2"
-					(reference "#PWR018")
+					(reference "#PWR012")
 					(unit 1)
 				)
@@
 		(dnp no)
 		(fields_autoplaced yes)
-		(property "Reference" "#PWR017"
+		(property "Reference" "#PWR011"
 			(at 19.05 142.24 0)
 			(hide yes)
@@
 			(project "Overkill-core"
 				(path "/fc53a0b2-7a4c-469b-8f54-4e370debb709/b418b60c-f580-4941-9de1-4c275543c012/c2c849f9-72ec-481b-977e-253b138385b2"
-					(reference "#PWR017")
+					(reference "#PWR011")
 					(unit 1)
 				)
@@
 		(dnp no)
 		(fields_autoplaced yes)
-		(property "Reference" "#PWR032"
+		(property "Reference" "#PWR026"
 			(at 270.51 138.43 0)
 			(hide yes)
@@
 			(project "Overkill-core"
 				(path "/fc53a0b2-7a4c-469b-8f54-4e370debb709/b418b60c-f580-4941-9de1-4c275543c012/c2c849f9-72ec-481b-977e-253b138385b2"
-					(reference "#PWR032")
+					(reference "#PWR026")
 					(unit 1)
 				)
@@
 		(dnp no)
 		(fields_autoplaced yes)
-		(property "Reference" "R22"
+		(property "Reference" "R18"
 			(at 266.7 20.32 90)
 			(show_name no)
@@
 			(project "Overkill-core"
 				(path "/fc53a0b2-7a4c-469b-8f54-4e370debb709/b418b60c-f580-4941-9de1-4c275543c012/c2c849f9-72ec-481b-977e-253b138385b2"
-					(reference "R22")
+					(reference "R18")
 					(unit 1)
 				)
@@
 		(dnp no)
 		(fields_autoplaced yes)
-		(property "Reference" "#PWR021"
+		(property "Reference" "#PWR015"
 			(at 74.93 49.53 0)
 			(hide yes)
@@
 			(project "Overkill-core"
 				(path "/fc53a0b2-7a4c-469b-8f54-4e370debb709/b418b60c-f580-4941-9de1-4c275543c012/c2c849f9-72ec-481b-977e-253b138385b2"
-					(reference "#PWR021")
+					(reference "#PWR015")
 					(unit 1)
 				)
@@
 		(dnp no)
 		(fields_autoplaced yes)
-		(property "Reference" "#PWR025"
+		(property "Reference" "#PWR019"
 			(at 177.8 161.29 0)
 			(hide yes)
@@
 			(project "Overkill-core"
 				(path "/fc53a0b2-7a4c-469b-8f54-4e370debb709/b418b60c-f580-4941-9de1-4c275543c012/c2c849f9-72ec-481b-977e-253b138385b2"
-					(reference "#PWR025")
+					(reference "#PWR019")
 					(unit 1)
 				)
@@
 		(dnp no)
 		(fields_autoplaced yes)
-		(property "Reference" "#PWR020"
+		(property "Reference" "#PWR014"
 			(at 44.45 161.29 0)
 			(hide yes)
@@
 			(project "Overkill-core"
 				(path "/fc53a0b2-7a4c-469b-8f54-4e370debb709/b418b60c-f580-4941-9de1-4c275543c012/c2c849f9-72ec-481b-977e-253b138385b2"
-					(reference "#PWR020")
+					(reference "#PWR014")
 					(unit 1)
 				)
@@
 		(dnp no)
 		(fields_autoplaced yes)
-		(property "Reference" "#PWR028"
+		(property "Reference" "#PWR022"
 			(at 214.63 92.71 0)
 			(hide yes)
@@
 			(project "Overkill-core"
 				(path "/fc53a0b2-7a4c-469b-8f54-4e370debb709/b418b60c-f580-4941-9de1-4c275543c012/c2c849f9-72ec-481b-977e-253b138385b2"
-					(reference "#PWR028")
+					(reference "#PWR022")
 					(unit 1)
 				)
@@
 		(dnp no)
 		(fields_autoplaced yes)
-		(property "Reference" "R20"
+		(property "Reference" "R16"
 			(at 245.11 126.9999 0)
 			(show_name no)
@@
 			(project "Overkill-core"
 				(path "/fc53a0b2-7a4c-469b-8f54-4e370debb709/b418b60c-f580-4941-9de1-4c275543c012/c2c849f9-72ec-481b-977e-253b138385b2"
-					(reference "R20")
+					(reference "R16")
 					(unit 1)
 				)
@@
 		(dnp no)
 		(fields_autoplaced yes)
-		(property "Reference" "#PWR019"
+		(property "Reference" "#PWR013"
 			(at 38.1 125.73 0)
 			(hide yes)
@@
 			(project "Overkill-core"
 				(path "/fc53a0b2-7a4c-469b-8f54-4e370debb709/b418b60c-f580-4941-9de1-4c275543c012/c2c849f9-72ec-481b-977e-253b138385b2"
-					(reference "#PWR019")
+					(reference "#PWR013")
 					(unit 1)
 				)
@@
 		(dnp no)
 		(fields_autoplaced yes)
-		(property "Reference" "R17"
+		(property "Reference" "R13"
 			(at 33.02 139.7 90)
 			(show_name no)
@@
 			(project "Overkill-core"
 				(path "/fc53a0b2-7a4c-469b-8f54-4e370debb709/b418b60c-f580-4941-9de1-4c275543c012/c2c849f9-72ec-481b-977e-253b138385b2"
-					(reference "R17")
+					(reference "R13")
 					(unit 1)
 				)
@@
 		(dnp no)
 		(fields_autoplaced yes)
-		(property "Reference" "R19"
+		(property "Reference" "R15"
 			(at 234.95 33.0199 0)
 			(show_name no)
@@
 			(project "Overkill-core"
 				(path "/fc53a0b2-7a4c-469b-8f54-4e370debb709/b418b60c-f580-4941-9de1-4c275543c012/c2c849f9-72ec-481b-977e-253b138385b2"
-					(reference "R19")
+					(reference "R15")
 					(unit 1)
 				)
@@
 		(dnp no)
 		(fields_autoplaced yes)
-		(property "Reference" "R21"
+		(property "Reference" "R17"
 			(at 250.19 33.0199 0)
 			(show_name no)
@@
 			(project "Overkill-core"
 				(path "/fc53a0b2-7a4c-469b-8f54-4e370debb709/b418b60c-f580-4941-9de1-4c275543c012/c2c849f9-72ec-481b-977e-253b138385b2"
-					(reference "R21")
+					(reference "R17")
 					(unit 1)
 				)
@@
 		(dnp no)
 		(fields_autoplaced yes)
-		(property "Reference" "#PWR027"
+		(property "Reference" "#PWR021"
 			(at 209.55 125.73 0)
 			(hide yes)
@@
 			(project "Overkill-core"
 				(path "/fc53a0b2-7a4c-469b-8f54-4e370debb709/b418b60c-f580-4941-9de1-4c275543c012/c2c849f9-72ec-481b-977e-253b138385b2"
-					(reference "#PWR027")
+					(reference "#PWR021")
 					(unit 1)
 				)
@@
 		(dnp no)
 		(fields_autoplaced yes)
-		(property "Reference" "U5"
+		(property "Reference" "U4"
 			(at 175.26 55.8098 0)
 			(show_name no)
@@
 			(project "Overkill-core"
 				(path "/fc53a0b2-7a4c-469b-8f54-4e370debb709/b418b60c-f580-4941-9de1-4c275543c012/c2c849f9-72ec-481b-977e-253b138385b2"
-					(reference "U5")
+					(reference "U4")
 					(unit 1)
 				)
@@
 		(dnp no)
 		(fields_autoplaced yes)
-		(property "Reference" "#PWR029"
+		(property "Reference" "#PWR023"
 			(at 242.57 53.34 0)
 			(hide yes)
@@
 			(project "Overkill-core"
 				(path "/fc53a0b2-7a4c-469b-8f54-4e370debb709/b418b60c-f580-4941-9de1-4c275543c012/c2c849f9-72ec-481b-977e-253b138385b2"
-					(reference "#PWR029")
+					(reference "#PWR023")
 					(unit 1)
 				)
@@
 		(dnp no)
 		(fields_autoplaced yes)
-		(property "Reference" "#PWR023"
+		(property "Reference" "#PWR017"
 			(at 152.4 49.53 0)
 			(hide yes)
@@
 			(project "Overkill-core"
 				(path "/fc53a0b2-7a4c-469b-8f54-4e370debb709/b418b60c-f580-4941-9de1-4c275543c012/c2c849f9-72ec-481b-977e-253b138385b2"
-					(reference "#PWR023")
+					(reference "#PWR017")
 					(unit 1)
 				)
@@
 		(dnp no)
 		(fields_autoplaced yes)
-		(property "Reference" "#PWR026"
+		(property "Reference" "#PWR020"
 			(at 196.85 107.95 0)
 			(hide yes)
@@
 			(project "Overkill-core"
 				(path "/fc53a0b2-7a4c-469b-8f54-4e370debb709/b418b60c-f580-4941-9de1-4c275543c012/c2c849f9-72ec-481b-977e-253b138385b2"
-					(reference "#PWR026")
+					(reference "#PWR020")
 					(unit 1)
 				)
@@
 		(dnp no)
 		(fields_autoplaced yes)
-		(property "Reference" "#PWR030"
+		(property "Reference" "#PWR024"
 			(at 256.54 161.29 0)
 			(hide yes)
@@
 			(project "Overkill-core"
 				(path "/fc53a0b2-7a4c-469b-8f54-4e370debb709/b418b60c-f580-4941-9de1-4c275543c012/c2c849f9-72ec-481b-977e-253b138385b2"
-					(reference "#PWR030")
+					(reference "#PWR024")
 					(unit 1)
 				)
