File: module.kicad_sch (KiCad schematic)
At the start: 2 parts

Commit message: updates
Parts:
- renumbered R25 to R21, R26 to R22
Changed lines of the file:
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@@
 		(dnp no)
 		(fields_autoplaced yes)
-		(property "Reference" "R26"
+		(property "Reference" "R22"
 			(at 172.72 111.7599 0)
 			(show_name no)
@@
 			(project "Overkill-core"
 				(path "/fc53a0b2-7a4c-469b-8f54-4e370debb709/b418b60c-f580-4941-9de1-4c275543c012"
-					(reference "R26")
+					(reference "R22")
 					(unit 1)
 				)
@@
 		(dnp no)
 		(fields_autoplaced yes)
-		(property "Reference" "#PWR037"
+		(property "Reference" "#PWR031"
 			(at 170.18 100.33 0)
 			(hide yes)
@@
 			(project "Overkill-core"
 				(path "/fc53a0b2-7a4c-469b-8f54-4e370debb709/b418b60c-f580-4941-9de1-4c275543c012"
-					(reference "#PWR037")
+					(reference "#PWR031")
 					(unit 1)
 				)
@@
 		(dnp no)
 		(fields_autoplaced yes)
-		(property "Reference" "R25"
+		(property "Reference" "R21"
 			(at 172.72 88.8999 0)
 			(show_name no)
@@
 			(project "Overkill-core"
 				(path "/fc53a0b2-7a4c-469b-8f54-4e370debb709/b418b60c-f580-4941-9de1-4c275543c012"
-					(reference "R25")
+					(reference "R21")
 					(unit 1)
 				)
@@
 		(dnp no)
 		(fields_autoplaced yes)
-		(property "Reference" "#PWR038"
+		(property "Reference" "#PWR032"
 			(at 170.18 123.19 0)
 			(hide yes)
@@
 			(project "Overkill-core"
 				(path "/fc53a0b2-7a4c-469b-8f54-4e370debb709/b418b60c-f580-4941-9de1-4c275543c012"
-					(reference "#PWR038")
-					(unit 1)
-				)
+					(reference "#PWR032")
+					(unit 1)
+				)
