File: p4_power.kicad_sch (KiCad schematic)
At the start: 11 parts, among them U7 MP1605GTF-Z

Commit message: updates
Parts:
- renumbered R23 to R19, R24 to R20, U7 to U6
Changed lines of the file:
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@@
 		(dnp no)
 		(fields_autoplaced yes)
-		(property "Reference" "#PWR036"
+		(property "Reference" "#PWR030"
 			(at 91.44 57.15 0)
 			(hide yes)
@@
 			(project "Overkill-core"
 				(path "/fc53a0b2-7a4c-469b-8f54-4e370debb709/b418b60c-f580-4941-9de1-4c275543c012/ee985d65-bcc1-4e4e-9738-4eeef2164bc1"
-					(reference "#PWR036")
+					(reference "#PWR030")
 					(unit 1)
 				)
@@
 		(dnp no)
 		(fields_autoplaced yes)
-		(property "Reference" "#PWR033"
+		(property "Reference" "#PWR027"
 			(at 25.4 50.8 0)
 			(hide yes)
@@
 			(project "Overkill-core"
 				(path "/fc53a0b2-7a4c-469b-8f54-4e370debb709/b418b60c-f580-4941-9de1-4c275543c012/ee985d65-bcc1-4e4e-9738-4eeef2164bc1"
-					(reference "#PWR033")
+					(reference "#PWR027")
 					(unit 1)
 				)
@@
 		(dnp no)
 		(fields_autoplaced yes)
-		(property "Reference" "U7"
+		(property "Reference" "U6"
 			(at 45.72 24.13 0)
 			(show_name no)
@@
 			(project "Overkill-core"
 				(path "/fc53a0b2-7a4c-469b-8f54-4e370debb709/b418b60c-f580-4941-9de1-4c275543c012/ee985d65-bcc1-4e4e-9738-4eeef2164bc1"
-					(reference "U7")
+					(reference "U6")
 					(unit 1)
 				)
@@
 		(dnp no)
 		(fields_autoplaced yes)
-		(property "Reference" "R24"
+		(property "Reference" "R20"
 			(at 71.12 53.3399 0)
 			(show_name no)
@@
 			(project "Overkill-core"
 				(path "/fc53a0b2-7a4c-469b-8f54-4e370debb709/b418b60c-f580-4941-9de1-4c275543c012/ee985d65-bcc1-4e4e-9738-4eeef2164bc1"
-					(reference "R24")
+					(reference "R20")
 					(unit 1)
 				)
@@
 		(dnp no)
 		(fields_autoplaced yes)
-		(property "Reference" "#PWR035"
+		(property "Reference" "#PWR029"
 			(at 68.58 64.77 0)
 			(hide yes)
@@
 			(project "Overkill-core"
 				(path "/fc53a0b2-7a4c-469b-8f54-4e370debb709/b418b60c-f580-4941-9de1-4c275543c012/ee985d65-bcc1-4e4e-9738-4eeef2164bc1"
-					(reference "#PWR035")
+					(reference "#PWR029")
 					(unit 1)
 				)
@@
 		(dnp no)
 		(fields_autoplaced yes)
-		(property "Reference" "#PWR034"
+		(property "Reference" "#PWR028"
 			(at 25.4 34.29 0)
 			(hide yes)
@@
 			(project "Overkill-core"
 				(path "/fc53a0b2-7a4c-469b-8f54-4e370debb709/b418b60c-f580-4941-9de1-4c275543c012/ee985d65-bcc1-4e4e-9738-4eeef2164bc1"
-					(reference "#PWR034")
+					(reference "#PWR028")
 					(unit 1)
 				)
@@
 		(dnp no)
 		(fields_autoplaced yes)
-		(property "Reference" "R23"
+		(property "Reference" "R19"
 			(at 71.12 45.7199 0)
 			(show_name no)
@@
 			(project "Overkill-core"
 				(path "/fc53a0b2-7a4c-469b-8f54-4e370debb709/b418b60c-f580-4941-9de1-4c275543c012/ee985d65-bcc1-4e4e-9738-4eeef2164bc1"
-					(reference "R23")
-					(unit 1)
-				)
+					(reference "R19")
+					(unit 1)
+				)
