File: power.kicad_sch (KiCad schematic)
At the start: 36 parts, among them Q1 BC808, Q2 BC808, Q3 BC808, Q4 BC808, Q5 AO3401A, Q6 AO3401A, U10 DIO7003HDST5, U11 AOZ1284PI

Commit message: updates
Parts:
- renumbered D4 to D2, R29 to R25, R30 to R26, R31 to R27, R32 to R28, R33 to R29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
