File: regulators.kicad_sch (KiCad schematic)
At the start: 12 parts, among them U8 TLV75733PDBV, U9 TLV75728PDBV

Commit message: updates
Parts:
- renumbered R27 to R23, R28 to R24, U8 to U7, U9 to U8
Changed lines of the file:
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@@
 		(dnp no)
 		(fields_autoplaced yes)
-		(property "Reference" "#PWR041"
+		(property "Reference" "#PWR035"
 			(at 63.5 49.53 0)
 			(hide yes)
@@
 			(project "Overkill-core"
 				(path "/fc53a0b2-7a4c-469b-8f54-4e370debb709/7d895a5c-8b95-494b-ac5d-52a816ea07bf"
-					(reference "#PWR041")
+					(reference "#PWR035")
 					(unit 1)
 				)
@@
 		(dnp no)
 		(fields_autoplaced yes)
-		(property "Reference" "#PWR042"
+		(property "Reference" "#PWR036"
 			(at 63.5 77.47 0)
 			(hide yes)
@@
 			(project "Overkill-core"
 				(path "/fc53a0b2-7a4c-469b-8f54-4e370debb709/7d895a5c-8b95-494b-ac5d-52a816ea07bf"
-					(reference "#PWR042")
+					(reference "#PWR036")
 					(unit 1)
 				)
@@
 		(dnp no)
 		(fields_autoplaced yes)
-		(property "Reference" "U9"
+		(property "Reference" "U8"
 			(at 63.5 52.07 0)
 			(show_name no)
@@
 			(project "Overkill-core"
 				(path "/fc53a0b2-7a4c-469b-8f54-4e370debb709/7d895a5c-8b95-494b-ac5d-52a816ea07bf"
-					(reference "U9")
+					(reference "U8")
 					(unit 1)
 				)
@@
 		(dnp no)
 		(fields_autoplaced yes)
-		(property "Reference" "#PWR043"
+		(property "Reference" "#PWR037"
 			(at 85.09 33.02 0)
 			(hide yes)
@@
 			(project "Overkill-core"
 				(path "/fc53a0b2-7a4c-469b-8f54-4e370debb709/7d895a5c-8b95-494b-ac5d-52a816ea07bf"
-					(reference "#PWR043")
+					(reference "#PWR037")
 					(unit 1)
 				)
@@
 		(dnp no)
 		(fields_autoplaced yes)
-		(property "Reference" "#PWR039"
+		(property "Reference" "#PWR033"
 			(at 25.4 33.02 0)
 			(hide yes)
@@
 			(project "Overkill-core"
 				(path "/fc53a0b2-7a4c-469b-8f54-4e370debb709/7d895a5c-8b95-494b-ac5d-52a816ea07bf"
-					(reference "#PWR039")
+					(reference "#PWR033")
 					(unit 1)
 				)
@@
 		(dnp no)
 		(fields_autoplaced yes)
-		(property "Reference" "R28"
+		(property "Reference" "R24"
 			(at 100.33 66.0399 0)
 			(show_name no)
@@
 			(project "Overkill-core"
 				(path "/fc53a0b2-7a4c-469b-8f54-4e370debb709/7d895a5c-8b95-494b-ac5d-52a816ea07bf"
-					(reference "R28")
+					(reference "R24")
 					(unit 1)
 				)
@@
 		(dnp no)
 		(fields_autoplaced yes)
-		(property "Reference" "R27"
+		(property "Reference" "R23"
 			(at 100.33 58.4199 0)
 			(show_name no)
@@
 			(project "Overkill-core"
 				(path "/fc53a0b2-7a4c-469b-8f54-4e370debb709/7d895a5c-8b95-494b-ac5d-52a816ea07bf"
-					(reference "R27")
+					(reference "R23")
 					(unit 1)
 				)
@@
 		(dnp no)
 		(fields_autoplaced yes)
-		(property "Reference" "#PWR046"
+		(property "Reference" "#PWR040"
 			(at 97.79 77.47 0)
 			(hide yes)
@@
 			(project "Overkill-core"
 				(path "/fc53a0b2-7a4c-469b-8f54-4e370debb709/7d895a5c-8b95-494b-ac5d-52a816ea07bf"
-					(reference "#PWR046")
+					(reference "#PWR040")
 					(unit 1)
 				)
@@
 		(dnp no)
 		(fields_autoplaced yes)
-		(property "Reference" "#PWR044"
+		(property "Reference" "#PWR038"
 			(at 85.09 60.96 0)
 			(hide yes)
@@
 			(project "Overkill-core"
 				(path "/fc53a0b2-7a4c-469b-8f54-4e370debb709/7d895a5c-8b95-494b-ac5d-52a816ea07bf"
-					(reference "#PWR044")
+					(reference "#PWR038")
 					(unit 1)
 				)
@@
 		(dnp no)
 		(fields_autoplaced yes)
-		(property "Reference" "#PWR040"
+		(property "Reference" "#PWR034"
 			(at 25.4 60.96 0)
 			(hide yes)
@@
 			(project "Overkill-core"
 				(path "/fc53a0b2-7a4c-469b-8f54-4e370debb709/7d895a5c-8b95-494b-ac5d-52a816ea07bf"
-					(reference "#PWR040")
+					(reference "#PWR034")
 					(unit 1)
 				)
@@
 		(dnp no)
 		(fields_autoplaced yes)
-		(property "Reference" "U8"
+		(property "Reference" "U7"
 			(at 63.5 24.13 0)
 			(show_name no)
@@
 			(project "Overkill-core"
 				(path "/fc53a0b2-7a4c-469b-8f54-4e370debb709/7d895a5c-8b95-494b-ac5d-52a816ea07bf"
-					(reference "U8")
+					(reference "U7")
 					(unit 1)
 				)
@@
 		(dnp no)
 		(fields_autoplaced yes)
-		(property "Reference" "#PWR045"
+		(property "Reference" "#PWR039"
 			(at 97.79 59.69 0)
 			(hide yes)
@@
 			(project "Overkill-core"
 				(path "/fc53a0b2-7a4c-469b-8f54-4e370debb709/7d895a5c-8b95-494b-ac5d-52a816ea07bf"
-					(reference "#PWR045")
-					(unit 1)
-				)
+					(reference "#PWR039")
+					(unit 1)
+				)
