File: usbuart.kicad_sch (KiCad schematic)
At the start: 33 parts, among them J10 USB_A, J11 USB_A, J4 Conn_01x03_Pin, J5 Conn_01x04_Pin, J6 Conn_01x02_Pin, J7 Conn_01x02_Pin, J8 USB_A, J9 USB_A, Q7 BC817, Q8 BC817, U1 CH343P, U12 CH334F, U13 FSUSB42MUX, Y4 12MHz

Commit message: updates
Parts:
- added D3, D4: SMF6V0A, Diode_SMD:D_SMF, symbol Diode:SMF6V0A
- added J2, J3: USB_C_Receptacle_USB2.0_14P, symbol Connector:USB_C_Receptacle_USB2.0_14P
- added R39, R40, R41, R42: 5.1k, symbol Device:R_Small_US
- renumbered C83 to C81, C81 to C83, C89 to C84, C88 to C85, C87 to C86, C85 to C87, C84 to C88, C86 to C89, J6 to J10, J7 to J11, J8 to J4, J9 to J5, J4 to J6, J10 to J7, J11 to J8, J5 to J9, R39 to R35, R40 to R36, R41 to R37, R42 to R38, U1 to U11
Connections:
- net USBHDS1_P is gone; now on net USBHSD1_P: U13.9 (HSD2+)
- net GND: now also D3.2 (A2), D4.2 (A2), J2.A1 (GND), J2.A12 (GND), J2.B1 (GND), J2.B12 (GND), J2.SH (SHIELD), J3.A1 (GND), J3.A12 (GND), J3.B1 (GND), J3.B12 (GND), J3.SH (SHIELD), R39.1, R40.1, R41.1, R42.1
- net USB0_5V: now also D3.1 (A1), J2.A4 (VBUS), J2.A9 (VBUS), J2.B4 (VBUS), J2.B9 (VBUS)
- net USB1_N: now also J4.2 (D-)
- net USB1_P: now also J4.3 (D+)
- net USB2_N: now also J5.2 (D-)
- net USB2_P: now also J5.3 (D+)
- net USB3_N: now also J7.2 (D-)
- net USB3_P: now also J7.3 (D+)
- net USBHSD1_N: now also J8.2 (D-)
- net USB_DBG_D_N: now also J2.A7 (D-), J2.B7 (D-)
- net USB_DBG_D_P: now also J2.A6 (D+), J2.B6 (D+)
- net VBUS_OUT: now also J4.1 (VBUS), J5.1 (VBUS), J7.1 (VBUS), J8.1 (VBUS)
- net USBHSD1_P: now reaches J8.3 (D+)
- new net: J3.B5 (CC2), R41.2
- new net: J2.A5 (CC1), R40.2
- new net: J2.B5 (CC2), R39.2
- new net: J3.A5 (CC1), R42.2
- new net USB1P1_N: J3.A7 (D-), J3.B7 (D-)
- new net USB1P1_P: J3.A6 (D+), J3.B6 (D+)
- new net USB1_5V: D4.1 (A1), J3.A4 (VBUS), J3.A9 (VBUS), J3.B4 (VBUS), J3.B9 (VBUS)
Other:
- moved on the sheet: C81, C82, C83, C84, C85, C86, C87, C88, C89, C91, D5, J10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
